File: eagle/attitude_driver/attitude_driver.sch (EAGLE design)
At the start: 28 parts, among them J1 BT-HC06, J10 ESC2-POWER, J11 ESC3-POWER, J12 SOURCE-POWER, J13 HALL-POWER, J14 PROGRAM, J17 CURRENT-SENSOR, J2 mpu9250, J3 ESC1-PWM, J4 ESC2-PWM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

Commit message: ordered components
Parts:
- removed J14: PROGRAM, SparkFun-Connectors:CONN_06LOCK_LONGPADS
- removed J2: mpu9250, SparkFun-Connectors:CONN_08LOCK_LONGPADS
- added U$4: WIRELESS-BLUETOOTH-HC-05-MIRRORMIRROR, diy-modules:WIRELESS-BLUETOOTH-HC-05-MIRRORMIRROR
- J1: value BT-HC06 -> (none); device SparkFun-Connectors:CONN_04LOCK_LONGPADS -> gy-91:GY-91LOCK_LONGPADS
Connections:
- net 3V3: now also J1.7; no longer J2.7
- net CSB: now also J1.1; no longer J2.1
- net ESC1-5V: now also J1.8, U$4.+5V; no longer J1.4, J2.8
- net GND: now also J1.6, U$4.GND; no longer J1.3, J14.1, J14.2, J2.6
- net N$1: now also U$4.RX; no longer J1.1
- net NCS: now also J1.2; no longer J2.2
- net PROG-5V: no longer J14.3
- net RST: no longer J14.6
- net RX: now also U$4.TX; no longer J1.2, J14.4
- net SAO: now also J1.3; no longer J2.3
- net SCL: now also J1.5; no longer J2.5
- net SDA: now also J1.4; no longer J2.4
- net TX: no longer J14.5
Changed lines of the file:
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@@
 <layer number="230" name="230bmp" color="7" fill="1" visible="yes" active="yes"/>
 <layer number="231" name="231bmp" color="7" fill="1" visible="yes" active="yes"/>
+<layer number="232" name="Eagle3D_PG2" color="7" fill="1" visible="yes" active="yes"/>
+<layer number="233" name="Eagle3D_PG3" color="7" fill="1" visible="yes" active="yes"/>
 <layer number="248" name="Housing" color="7" fill="1" visible="yes" active="yes"/>
 <layer number="249" name="Edge" color="7" fill="1" visible="yes" active="yes"/>
@@
 <parts>
 <part name="B1" library="SparkFun-Boards" deviceset="ARDUINO_PRO_MINI" device=""/>
-<part name="J2" library="SparkFun-Connectors" deviceset="CONN_08" device="LOCK_LONGPADS" value="mpu9250"/>
 <part name="J3" library="SparkFun-Connectors" deviceset="CONN_03" device="LOCK_LONGPADS" value="ESC1-PWM"/>
 <part name="J4" library="SparkFun-Connectors" deviceset="CONN_03" device="LOCK_LONGPADS" value="ESC2-PWM"/>
@@
 <part name="J12" library="SparkFun-Connectors" deviceset="CONN_02" device="LOCK_LONGPADS" value="SOURCE-POWER"/>
 <part name="J13" library="SparkFun-Connectors" deviceset="CONN_02" device="LOCK_LONGPADS" value="HALL-POWER"/>
-<part name="J1" library="SparkFun-Connectors" deviceset="CONN_04" device="LOCK_LONGPADS" value="BT-HC06"/>
-<part name="J14" library="SparkFun-Connectors" deviceset="CONN_06" device="LOCK_LONGPADS" value="PROGRAM"/>
 <part name="R2" library="resistors-longpads" deviceset="1KOHM" device="-HORIZ-1/4W-5%" value="1k"/>
 <part name="R1" library="resistors-longpads" deviceset="RESISTOR" device="AXIAL-0.3" value="2k"/>
@@
 <part name="R3" library="SparkFun-Resistors" deviceset="1KOHM" device="-HORIZ-1/4W-1%" value="1k"/>
 <part name="D2" library="SparkFun-DiscreteSemi" deviceset="DIODE" device="-1N4148" value="200mA/100V/1V"/>
+<part name="J1" library="gy-91" deviceset="GY-91" device="LOCK_LONGPADS"/>
+<part name="U$4" library="diy-modules" deviceset="WIRELESS-BLUETOOTH-HC-05-MIRROR" device="MIRROR"/>
 </parts>
 <sheets>
@@
 <instances>
 <instance part="B1" gate="G$1" x="20.32" y="38.1"/>
-<instance part="J2" gate="G$1" x="-76.2" y="15.24"/>
 <instance part="J3" gate="J$1" x="60.96" y="58.42"/>
 <instance part="J4" gate="J$1" x="60.96" y="40.64"/>
@@
 <instance part="J12" gate="G$1" x="88.9" y="27.94" rot="R270"/>
 <instance part="J13" gate="G$1" x="-33.02" y="33.02"/>
-<instance part="J1" gate="G$1" x="-76.2" y="50.8"/>
-<instance part="J14" gate="G$1" x="20.32" y="81.28" rot="R270"/>
 <instance part="R2" gate="G$1" x="-55.88" y="48.26"/>
 <instance part="R1" gate="G$1" x="-63.5" y="40.64" rot="R90"/>
@@
 <instance part="R3" gate="G$1" x="101.6" y="104.14"/>
 <instance part="D2" gate="G$1" x="91.44" y="104.14"/>
+<instance part="J1" gate="G$1" x="-76.2" y="15.24"/>
+<instance part="U$4" gate="G$1" x="-91.44" y="50.8" rot="R180"/>
 </instances>
 <busses>
@@
 <pinref part="R1" gate="G$1" pin="2"/>
 <wire x1="-63.5" y1="48.26" x2="-63.5" y2="45.72" width="0.1524" layer="91"/>
-<pinref part="J1" gate="G$1" pin="1"/>
 <wire x1="-71.12" y1="48.26" x2="-63.5" y2="48.26" width="0.1524" layer="91"/>
 <junction x="-63.5" y="48.26"/>
+<pinref part="U$4" gate="G$1" pin="RX"/>
 </segment>
 </net>
@@
 <label x="2.54" y="55.88" size="1.778" layer="95"/>
 </segment>
-<segment>
-<pinref part="J14" gate="G$1" pin="5"/>
-<wire x1="25.4" y1="76.2" x2="25.4" y2="73.66" width="0.1524" layer="91"/>
-<label x="25.4" y="71.12" size="1.778" layer="95" rot="R90"/>
-</segment>
 </net>
 <net name="GND" class="0">
@@
 </segment>
 <segment>
-<pinref part="J1" gate="G$1" pin="3"/>
 <wire x1="-71.12" y1="53.34" x2="-68.58" y2="53.34" width="0.1524" layer="91"/>
 <label x="-68.58" y="53.34" size="1.778" layer="95"/>
-</segment>
-<segment>
-<pinref part="J2" gate="G$1" pin="6"/>
+<pinref part="U$4" gate="G$1" pin="GND"/>
+</segment>
+<segment>
 <wire x1="-71.12" y1="20.32" x2="-68.58" y2="20.32" width="0.1524" layer="91"/>
 <label x="-68.58" y="20.32" size="1.778" layer="95"/>
+<pinref part="J1" gate="G$1" pin="6"/>
 </segment>
 <segment>
@@
 <pinref part="J11" gate="G$1" pin="2"/>
 <wire x1="137.16" y1="-2.54" x2="137.16" y2="20.32" width="0.1524" layer="91"/>
-</segment>
-<segment>
-<pinref part="J14" gate="G$1" pin="1"/>
-<wire x1="15.24" y1="76.2" x2="15.24" y2="73.66" width="0.1524" layer="91"/>
-<label x="15.24" y="71.12" size="1.778" layer="95" rot="R90"/>
-</segment>
-<segment>
-<pinref part="J14" gate="G$1" pin="2"/>
-<wire x1="17.78" y1="76.2" x2="17.78" y2="73.66" width="0.1524" layer="91"/>
-<label x="17.78" y="71.12" size="1.778" layer="95" rot="R90"/>
 </segment>
 <segment>
@@
 <net name="RX" class="0">
 <segment>
-<pinref part="J1" gate="G$1" pin="2"/>
 <wire x1="-71.12" y1="50.8" x2="-68.58" y2="50.8" width="0.1524" layer="91"/>
 <label x="-68.58" y="50.8" size="1.778" layer="95"/>
+<pinref part="U$4" gate="G$1" pin="TX"/>
 </segment>
 <segment>
@@
 <label x="2.54" y="53.34" size="1.778" layer="95"/>
 </segment>
-<segment>
-<pinref part="J14" gate="G$1" pin="4"/>
-<wire x1="22.86" y1="76.2" x2="22.86" y2="73.66" width="0.1524" layer="91"/>
-<label x="22.86" y="71.12" size="1.778" layer="95" rot="R90"/>
-</segment>
 </net>
 <net name="3V3" class="0">
 <segment>
-<pinref part="J2" gate="G$1" pin="7"/>
 <wire x1="-71.12" y1="22.86" x2="-68.58" y2="22.86" width="0.1524" layer="91"/>
 <label x="-68.58" y="22.86" size="1.778" layer="95"/>
+<pinref part="J1" gate="G$1" pin="7"/>
 </segment>
 </net>
 <net name="SCL" class="0">
 <segment>
-<pinref part="J2" gate="G$1" pin="5"/>
 <wire x1="-71.12" y1="17.78" x2="-68.58" y2="17.78" width="0.1524" layer="91"/>
 <label x="-68.58" y="17.78" size="1.778" layer="95"/>
+<pinref part="J1" gate="G$1" pin="5"/>
 </segment>
 <segment>
@@
 <net name="SDA" class="0">
 <segment>
-<pinref part="J2" gate="G$1" pin="4"/>
 <wire x1="-71.12" y1="15.24" x2="-68.58" y2="15.24" width="0.1524" layer="91"/>
 <label x="-68.58" y="15.24" size="1.778" layer="95"/>
+<pinref part="J1" gate="G$1" pin="4"/>
 </segment>
 <segment>
@@
 <net name="SAO" class="0">
 <segment>
-<pinref part="J2" gate="G$1" pin="3"/>
 <wire x1="-71.12" y1="12.7" x2="-68.58" y2="12.7" width="0.1524" layer="91"/>
 <label x="-68.58" y="12.7" size="1.778" layer="95"/>
+<pinref part="J1" gate="G$1" pin="3"/>
 </segment>
 <segment>
@@
 <net name="NCS" class="0">
 <segment>
-<pinref part="J2" gate="G$1" pin="2"/>
 <wire x1="-71.12" y1="10.16" x2="-68.58" y2="10.16" width="0.1524" layer="91"/>
 <label x="-68.58" y="10.16" size="1.778" layer="95"/>
+<pinref part="J1" gate="G$1" pin="2"/>
 </segment>
 <segment>
@@
 <net name="CSB" class="0">
 <segment>
-<pinref part="J2" gate="G$1" pin="1"/>
 <wire x1="-71.12" y1="7.62" x2="-68.58" y2="7.62" width="0.1524" layer="91"/>
 <label x="-68.58" y="7.62" size="1.778" layer="95"/>
+<pinref part="J1" gate="G$1" pin="1"/>
 </segment>
 <segment>
@@
 </segment>
 <segment>
-<pinref part="J2" gate="G$1" pin="8"/>
 <wire x1="-71.12" y1="25.4" x2="-68.58" y2="25.4" width="0.1524" layer="91"/>
 <label x="-68.58" y="25.4" size="1.778" layer="95"/>
-</segment>
-<segment>
-<pinref part="J1" gate="G$1" pin="4"/>
+<pinref part="J1" gate="G$1" pin="8"/>
+</segment>
+<segment>
 <wire x1="-71.12" y1="55.88" x2="-68.58" y2="55.88" width="0.1524" layer="91"/>
 <label x="-68.58" y="55.88" size="1.778" layer="95"/>
+<pinref part="U$4" gate="G$1" pin="+5V"/>
 </segment>
 <segment>
@@
 <wire x1="10.16" y1="50.8" x2="7.62" y2="50.8" width="0.1524" layer="91"/>
 <label x="2.54" y="50.8" size="1.778" layer="95"/>
-</segment>
-<segment>
-<pinref part="J14" gate="G$1" pin="6"/>
-<wire x1="27.94" y1="76.2" x2="27.94" y2="73.66" width="0.1524" layer="91"/>
-<label x="27.94" y="71.12" size="1.778" layer="95" rot="R90"/>
 </segment>
 </net>
@@
 <label x="43.18" y="66.04" size="1.778" layer="95" rot="R90"/>
 </segment>
-<segment>
-<pinref part="J14" gate="G$1" pin="3"/>
-<wire x1="20.32" y1="76.2" x2="20.32" y2="73.66" width="0.1524" layer="91"/>
-<label x="20.32" y="71.12" size="1.778" layer="95" rot="R90"/>
-</segment>
-</net>
+</net>

Commit message: update pcb design
Connections:
- new net N$4: D1.C, T1.E, U$1.COIL0, U$2.COIL1
- net ESC2-5V: no longer J16.1
- net ESC3-5V: now also J16.1
- net GND: no longer D1.C, T1.E, U$1.COIL0, U$2.COIL1
Changed lines of the file:
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@@
 <setting verticaltext="up"/>
 </settings>
-<grid distance="0.1" unitdist="inch" unit="mm" style="dots" multiple="1" display="yes" altdistance="0.01" altunitdist="inch" altunit="mm"/>
+<grid distance="0.1" unitdist="inch" unit="inch" style="lines" multiple="1" display="no" altdistance="0.01" altunitdist="inch" altunit="inch"/>
 <layers>
 <layer number="1" name="Top" color="4" fill="1" visible="no" active="no"/>
@@
 </variantdefs>
 <classes>
-<class number="0" name="default" width="0" drill="0">
+<class number="0" name="default" width="1" drill="0">
+<clearance class="0" value="0.3"/>
 </class>
 </classes>
@@
 </segment>
 <segment>
-<pinref part="U$1" gate="G$1" pin="COIL0"/>
-<pinref part="U$2" gate="G$1" pin="COIL1"/>
-<wire x1="127" y1="88.9" x2="119.38" y2="88.9" width="0.1524" layer="91"/>
-<pinref part="T1" gate="G$1" pin="E"/>
-<wire x1="119.38" y1="88.9" x2="111.76" y2="88.9" width="0.1524" layer="91"/>
-<wire x1="119.38" y1="99.06" x2="119.38" y2="88.9" width="0.1524" layer="91"/>
-<junction x="119.38" y="88.9"/>
-<pinref part="D1" gate="G$1" pin="C"/>
-<wire x1="119.38" y1="86.36" x2="119.38" y2="88.9" width="0.1524" layer="91"/>
-</segment>
-<segment>
 <pinref part="U$1" gate="G$1" pin="COIL1"/>
 <pinref part="U$2" gate="G$1" pin="COIL0"/>
@@
 <label x="71.12" y="40.64" size="1.778" layer="95"/>
 </segment>
+</net>
+<net name="ESC-S3" class="0">
+<segment>
+<pinref part="J5" gate="J$1" pin="3"/>
+<wire x1="68.58" y1="25.4" x2="71.12" y2="25.4" width="0.1524" layer="91"/>
+<label x="71.12" y="25.4" size="1.778" layer="95"/>
+</segment>
+<segment>
+<pinref part="B1" gate="G$1" pin="*9"/>
+<wire x1="10.16" y1="27.94" x2="7.62" y2="27.94" width="0.1524" layer="91"/>
+<label x="2.54" y="27.94" size="1.778" layer="95"/>
+</segment>
+</net>
+<net name="ESC3-5V" class="0">
+<segment>
+<pinref part="J5" gate="J$1" pin="2"/>
+<wire x1="68.58" y1="22.86" x2="71.12" y2="22.86" width="0.1524" layer="91"/>
+<label x="71.12" y="22.86" size="1.778" layer="95"/>
+</segment>
 <segment>
 <pinref part="J16" gate="G$1" pin="1"/>
 <wire x1="-25.4" y1="76.2" x2="-25.4" y2="73.66" width="0.1524" layer="91"/>
 <label x="-25.4" y="73.66" size="1.778" layer="95" rot="R270"/>
-</segment>
-</net>
-<net name="ESC-S3" class="0">
-<segment>
-<pinref part="J5" gate="J$1" pin="3"/>
-<wire x1="68.58" y1="25.4" x2="71.12" y2="25.4" width="0.1524" layer="91"/>
-<label x="71.12" y="25.4" size="1.778" layer="95"/>
-</segment>
-<segment>
-<pinref part="B1" gate="G$1" pin="*9"/>
-<wire x1="10.16" y1="27.94" x2="7.62" y2="27.94" width="0.1524" layer="91"/>
-<label x="2.54" y="27.94" size="1.778" layer="95"/>
-</segment>
-</net>
-<net name="ESC3-5V" class="0">
-<segment>
-<pinref part="J5" gate="J$1" pin="2"/>
-<wire x1="68.58" y1="22.86" x2="71.12" y2="22.86" width="0.1524" layer="91"/>
-<label x="71.12" y="22.86" size="1.778" layer="95"/>
 </segment>
 </net>
@@
 </segment>
 </net>
+<net name="N$4" class="0">
+<segment>
+<pinref part="U$1" gate="G$1" pin="COIL0"/>
+<pinref part="U$2" gate="G$1" pin="COIL1"/>
+<wire x1="111.76" y1="88.9" x2="119.38" y2="88.9" width="0.1524" layer="91"/>
+<pinref part="D1" gate="G$1" pin="C"/>
+<wire x1="119.38" y1="88.9" x2="127" y2="88.9" width="0.1524" layer="91"/>
+<wire x1="119.38" y1="86.36" x2="119.38" y2="88.9" width="0.1524" layer="91"/>
+<junction x="119.38" y="88.9"/>
+<pinref part="T1" gate="G$1" pin="E"/>
+<wire x1="119.38" y1="99.06" x2="119.38" y2="88.9" width="0.1524" layer="91"/>
+</segment>
+</net>
